Commit message: noetic-devel first commit

File: husky_ur3_gazebo/urdf/accessories/sick_tim571.urdf.xacro (robot description, xacro)
@@ -33,5 +33,5 @@
     <link name="${prefix}_link">
     </link>
-    <sensor_sick_tim571_gazebo/>
+    <xacro:sensor_sick_tim571_gazebo/>
   </xacro:macro>
   <xacro:macro name="sensor_sick_tim571_gazebo">
@@ -44,5 +44,5 @@
 					<scan>
 						<horizontal>
-							<samples>819</samples>
+							<samples>716</samples>
 							<resolution>1</resolution>
 							<min_angle>${min_angle}</min_angle>

File: husky_ur3_gazebo/urdf/decorations.urdf.xacro (robot description, xacro)
@@ -206,7 +206,7 @@
         <child link="mount_link"/>
     </joint>-->
-    <h_sensor_d435 parent="top_plate_link">
+    <xacro:h_sensor_d435 parent="top_plate_link">
         <origin xyz="0.4 0.0 0.06" rpy="0 0 0"/>
-    </h_sensor_d435>
+    </xacro:h_sensor_d435>
   </xacro:macro>
 </robot>

File: husky_ur3_gazebo/urdf/husky.urdf.xacro (robot description, xacro)
@@ -36,5 +36,5 @@
   <xacro:include filename="$(find husky_ur3_gazebo)/urdf/accessories/kinect_camera.urdf.xacro"/>
   <xacro:include filename="$(find husky_ur3_gazebo)/urdf/accessories/sick_lms1xx_mount.urdf.xacro"/>
-   <xacro:include filename="$(find husky_ur3_gazebo)/urdf/accessories/sick_tim571.urdf.xacro"/>
+  <xacro:include filename="$(find husky_ur3_gazebo)/urdf/accessories/sick_tim571.urdf.xacro"/>
   <xacro:include filename="$(find husky_ur3_gazebo)/urdf/accessories/sensor_arch.urdf.xacro"/>
   <xacro:include filename="$(find husky_ur3_gazebo)/urdf/ur3_robot.urdf.xacro"/>
@@ -155,4 +155,7 @@
    	<origin xyz="$(arg laser_xyz)" rpy="$(arg laser_rpy)"/>
   </xacro:sensor_sick_tim571>
+  <xacro:sensor_sick_tim571_gazebo prefix="front_laser">
+   	<origin xyz="$(arg laser_xyz)" rpy="$(arg laser_rpy)"/>
+  </xacro:sensor_sick_tim571_gazebo>
   <xacro:if value="$(arg kinect_enabled)">
     <xacro:sensor_arch prefix="" parent="top_plate_link">

File: husky_ur3_gazebo/urdf/husky_ur3_gripper.urdf.xacro (robot description, xacro)
@@ -24,10 +24,14 @@
   <xacro:arg name="laser_xyz" default="$(optenv HUSKY_LMS1XX_XYZ 0.3206 0.0 -0.000635)" />
   <xacro:arg name="laser_rpy" default="$(optenv HUSKY_LMS1XX_RPY 0.0 0 0)" />
-  <xacro:arg name="camera_h_enabled" default="false" />
-  <xacro:arg name="camera_g_enabled" default="false" />
-  <xacro:arg name="camera_h_xyz" default="$(optenv HUSKY_KINECT_XYZ 0 0 0)" />
-  <xacro:arg name="camera_h_rpy" default="$(optenv HUSKY_KINECT_RPY 0 0.18 3.14)" />
-  <xacro:arg name="camera_g_xyz" default="$(optenv HUSKY_KINECT_XYZ 0 0 0.1)" />
-  <xacro:arg name="camera_g_rpy" default="$(optenv HUSKY_KINECT_RPY 0 0.18 3.14)" />
+  <!-- camera_h: decorations.urdf.xacro -->
+  <!-- camera_g: ur3_robot_gripper.urdf.xacro -->
+  <!--
+  <xacro:arg name="camera_h_enabled" default="true" />
+  <xacro:arg name="camera_g_enabled" default="true" />
+  <xacro:arg name="camera_h_xyz" default="$(optenv HUSKY_KINECT_XYZ 0.33 0 0.01)" />
+  <xacro:arg name="camera_h_rpy" default="$(optenv HUSKY_KINECT_RPY 0 -0.314 0)" />
+  <xacro:arg name="camera_g_xyz" default="$(optenv HUSKY_KINECT_XYZ 0 0 0.04)" />
+  <xacro:arg name="camera_g_rpy" default="$(optenv HUSKY_KINECT_RPY 0 0 0)" />
+  -->
   <xacro:property name="husky_front_bumper_extend" value="$(optenv HUSKY_FRONT_BUMPER_EXTEND 0)" />
   <xacro:property name="husky_rear_bumper_extend" value="$(optenv HUSKY_REAR_BUMPER_EXTEND 0)" />
@@ -37,8 +41,9 @@
   <xacro:include filename="$(find husky_ur3_gazebo)/urdf/decorations.urdf.xacro" />
   <xacro:include filename="$(find husky_ur3_gazebo)/urdf/wheel.urdf.xacro" />
-  <xacro:include filename="$(find husky_ur3_gazebo)/urdf/accessories/sick_lms1xx_mount.urdf.xacro"/>
+  <xacro:include filename="$(find husky_ur3_gazebo)/urdf/accessories/sensor_arch.urdf.xacro"/>
   <xacro:include filename="$(find husky_ur3_gazebo)/urdf/accessories/sick_tim571.urdf.xacro"/>
   <xacro:include filename="$(find husky_ur3_gazebo)/urdf/ur3_robot_gripper.urdf.xacro"/>
   <xacro:include filename="$(find husky_ur3_gazebo)/urdf/accessories/d435_camera_h.urdf.xacro"/>-
+  <xacro:include filename="$(find husky_ur3_gazebo)/urdf/accessories/d435_camera_g.urdf.xacro"/>-
   <!--xacro:include filename="$(find husky_ur3_gazebo)/urdf/ur3_robot.urdf.xacro"/-->
   <xacro:property name="M_PI" value="3.14159"/>
@@ -158,22 +163,13 @@
    	<origin xyz="$(arg laser_xyz)" rpy="$(arg laser_rpy)"/>
   </xacro:sensor_sick_tim571>
-  <!--<xacro:if value="$(arg camera_h_enabled)">
-    <xacro:sensor_arch prefix="" parent="top_plate_link">
-      <origin xyz="0.4 0 0.0" rpy="0 0.50 -3.14"/>
-    </xacro:sensor_arch>
-    <joint name="h_camera_joint" type="fixed">
-      <origin xyz="$(arg camera_h_xyz)" rpy="$(arg camera_h_rpy)" />
-      <parent link="top_plate_link"/>
-      <child link="h_camera_link"/>
-    </joint>
-    <xacro:h_sensor_d435 prefix="h_camera" robot_namespace="$(arg robot_namespace)"/>
-  </xacro:if>-->
-  <!--<xacro:if value="$(arg camera_g_enabeld)">
-    <joint name="g_camera_joint" type="fixed">
+<!--  <xacro:if value="$(arg camera_h_enabled)">
+    <xacro:h_sensor_d435 parent="top_plate_link">
+      <origin xyz="$(arg camera_h_xyz)" rpy="$(arg camera_h_rpy)"/>
+    </xacro:h_sensor_d435>
+  </xacro:if>
+  <xacro:if value="$(arg camera_g_enabled)">
+    <xacro:g_sensor_d435 parent="ee_link">
       <origin xyz="$(arg camera_g_xyz)" rpy="$(arg camera_g_rpy)"/>
-      <parent link="ee_link"/>
-      <child link="g_camera_link"/>
-    </joint>
-    <xacro:g_sensor_d435 prefix="g_camera" robot_namespace="$(arg robot_namespace)"/>
+    </xacro:g_sensor_d435>
   </xacro:if>
 -->

File: husky_ur3_gazebo/urdf/ur3_robot_gripper.urdf.xacro (robot description, xacro)
@@ -29,6 +29,6 @@
           <origin xyz="0 0 0" rpy="0 1.57 0"/>
   </joint>
-  <g_sensor_d435 parent="ee_link">
+  <xacro:g_sensor_d435 parent="ee_link">
         <origin xyz="0.0 0.00 -0.04" rpy="${-pi} 0 0"/>
-    </g_sensor_d435>
+  </xacro:g_sensor_d435>
 </robot>
