Commit message: Update husky_ur3_gripper.urdf.xacro

File: husky_ur3_gazebo/urdf/husky_ur3_gripper.urdf.xacro (robot description, xacro)
@@ -163,15 +163,4 @@
    	<origin xyz="$(arg laser_xyz)" rpy="$(arg laser_rpy)"/>
   </xacro:sensor_sick_tim571>
-<!--  <xacro:if value="$(arg camera_h_enabled)">
-    <xacro:h_sensor_d435 parent="top_plate_link">
-      <origin xyz="$(arg camera_h_xyz)" rpy="$(arg camera_h_rpy)"/>
-    </xacro:h_sensor_d435>
-  </xacro:if>
-  <xacro:if value="$(arg camera_g_enabled)">
-    <xacro:g_sensor_d435 parent="ee_link">
-      <origin xyz="$(arg camera_g_xyz)" rpy="$(arg camera_g_rpy)"/>
-    </xacro:g_sensor_d435>
-  </xacro:if>
--->
  <joint name="control_box_ur3_joint" type="fixed">
       <origin xyz="-0.095 0 0.233" rpy="${M_PI/2} 0 0" />

Commit message: Update husky_ur3_gripper.urdf.xacro
remove some annotations because there was an error.

File: husky_ur3_gazebo/urdf/husky_ur3_gripper.urdf.xacro (robot description, xacro)
@@ -158,24 +158,4 @@
    	<origin xyz="$(arg laser_xyz)" rpy="$(arg laser_rpy)"/>
   </xacro:sensor_sick_tim571>
-  <!--<xacro:if value="$(arg camera_h_enabled)">
-    <xacro:sensor_arch prefix="" parent="top_plate_link">
-      <origin xyz="0.4 0 0.0" rpy="0 0.50 -3.14"/>
-    </xacro:sensor_arch>
-    <joint name="h_camera_joint" type="fixed">
-      <origin xyz="$(arg camera_h_xyz)" rpy="$(arg camera_h_rpy)" />
-      <parent link="top_plate_link"/>
-      <child link="h_camera_link"/>
-    </joint>
-    <xacro:h_sensor_d435 prefix="h_camera" robot_namespace="$(arg robot_namespace)"/>
-  </xacro:if>-->
-  <!--<xacro:if value="$(arg camera_g_enabeld)">
-    <joint name="g_camera_joint" type="fixed">
-      <origin xyz="$(arg camera_g_xyz)" rpy="$(arg camera_g_rpy)"/>
-      <parent link="ee_link"/>
-      <child link="g_camera_link"/>
-    </joint>
-    <xacro:g_sensor_d435 prefix="g_camera" robot_namespace="$(arg robot_namespace)"/>
-  </xacro:if>
--->
  <joint name="control_box_ur3_joint" type="fixed">
       <origin xyz="-0.095 0 0.233" rpy="${M_PI/2} 0 0" />
